File: cdm_exg_v1.kicad_pcb (KiCad board)
At the start: 4 copper layers, 271.8 x 195.6 mm, 278 parts, among them J1 SMA-OSU_SIM_BASIC, J10 Conn_01x02, J11 Conn_01x02, J12 SMA_5p5, J13 Conn_01x02, J14 Conn_01x02, J15 SMA-OSU_SIM_BASIC, J16 SMA-OSU_SIM_BASIC, J17 SMA-OSU_SIM_BASIC, J18 SMA-OSU_SIM_BASIC, J19 SMA-OSU_SIM_BASIC, J2 SMA-OSU_SIM_BASIC, J20 SMA-OSU_SIM_BASIC, J21 SMA-OSU_SIM_BASIC, J22 SMA-OSU_SIM_BASIC, J23 Conn_01x02, J24 Conn_01x02, J25 Conn_01x02, J26 Conn_01x02, J27 Conn_01x02, J28 Conn_01x02, J29 Conn_01x02, J3 SMA-OSU_SIM_BASIC, J30 Conn_01x02, J31 Conn_01x02, J32 Conn_01x02, J33 SMA-OSU_SIM_BASIC, J34 Conn_01x02, J35 SMA-OSU_SIM_BASIC, J36 Conn_01x01, J37 SMA-OSU_SIM_BASIC, J38 SMA-OSU_SIM_BASIC, J39 OPAL_KELLY, J4 SMA-OSU_SIM_BASIC, J40 SMA-OSU_SIM_BASIC, J41 Conn_01x01, J42 Conn_01x03, J43 Conn_01x03, J44 Conn_01x03, J45 Conn_01x01, J46 Conn_01x01, J47 Conn_01x01, J48 SMA-OSU_SIM_BASIC, J49 SMA-OSU_SIM_BASIC, J5 SMA-OSU_SIM_BASIC, J50 Conn_01x10, J51 Conn_01x02, J52 Conn_01x02, J53 Conn_01x02, J54 Conn_01x02, J55 Conn_01x02, J56 Conn_01x02, J57 Conn_01x02, J58 Conn_01x02, J59 Conn_01x01, J6 SMA-OSU_SIM_BASIC, J60 SMA-OSU_SIM_BASIC, J61 SMA-OSU_SIM_BASIC, J62 Conn_01x01, J63 Conn_01x03, J64 Conn_01x03, J65 Conn_01x01, J66 Conn_01x01, J67 Conn_01x01, J68 Conn_01x10, J69 Conn_01x02, J7 SMA-OSU_SIM_BASIC, J70 Conn_01x02, J71 Conn_01x02, J72 Conn_01x02, J73 Conn_01x02, J74 Conn_01x02, J75 Conn_01x02, J76 Conn_01x02, J77 Conn_01x02, J78 Conn_01x02, J79 Conn_01x02, J8 Conn_01x02, J80 Conn_01x02, J81 Conn_01x02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

Commit message: Feb20 commit
Parts:
- moved J44 16.7 mm to (92.3, 105.5)
- moved J87 16.2 mm to (103.0, 120.3)
Routing:
- net /AE_CHIP1/VCM_BE: track 58.7 -> 37.5 mm
- net /PVDD: track 136.0 -> 152.0 mm
- net /AE_CHIP1/ON_CHIP_TEST: track 18.6 -> 33.9 mm, vias 0 -> 1
- net /AE_CHIP1/VCM_AE: track 94.6 -> 83.8 mm
- net /AE_CHIP1/ADC_IP_BUF: vias 0 -> 1
Other:
- net class Default: trace_width 0.762 -> 0.508
